File: PCB/GanJing 65 rev 2.sch (KiCad schematic (older format))
At the start: 149 parts, among them SW1 EC11_rotary_encoder, U1 Elite-C

Commit message: Finished routing
Parts:
- added MX76: MX_1u_no_LED, GanJing_components:MX_1u_no_LED, symbol GanJing_components:MX_1u_no_LED
Connections:
- net S1: now also U1.14 (B4), MX76.1 (COL); no longer U1.13 (B5)
- net S2: now also MX76.2 (ROW)
- net col_1: now also U1.5 (F4); no longer U1.1 (B0)
- net col_10: now also U1.26 (F1); no longer U1.25 (F0)
- net col_11: now also U1.27 (C7); no longer U1.26 (F1)
- net col_12: now also U1.28 (D5); no longer U1.27 (C7)
- net col_13: now also U1.29 (B7); no longer U1.28 (D5)
- net col_14: now also U1.13 (B5); no longer U1.29 (B7)
- net col_2: now also U1.6 (F5); no longer U1.5 (F4)
- net col_3: now also U1.7 (F6); no longer U1.6 (F5)
- net col_4: now also U1.8 (F7); no longer U1.7 (F6)
- net col_5: now also U1.9 (B1/SCLK); no longer U1.8 (F7)
- net col_6: now also U1.10 (B3/MISO); no longer U1.9 (B1/SCLK)
- net col_7: now also U1.11 (B2/MOSI); no longer U1.10 (B3/MISO)
- net col_8: now also U1.12 (B6); no longer U1.11 (B2/MOSI)
- net col_9: now also U1.25 (F0); no longer U1.12 (B6)
- net row_1: now also U1.1 (B0); no longer U1.14 (B4)
Changed lines of the file:
@@
 Wire Wire Line
 	4000 6950 3950 6950
-Text GLabel 10450 1850 0    50   Input ~ 0
+Text GLabel 10550 1850 2    50   Input ~ 0
 S1
-Text GLabel 10300 2000 2    50   Input ~ 0
+Text GLabel 10550 2050 2    50   Input ~ 0
 S2
-Wire Wire Line
-	10300 2000 10250 2000
-Wire Wire Line
-	10250 2000 10250 2050
 $Comp
 L GanJing_components:1N4148TR_diode D71
@@
 	2150 3150 2150 3100
 Wire Wire Line
-	2050 3150 2050 3100
+	1500 2000 1550 2000
 Wire Wire Line
 	1500 2700 1550 2700
@@
 	1500 2200 1550 2200
 Wire Wire Line
+	1500 1900 1550 1900
+Wire Wire Line
+	1500 1600 1550 1600
+Wire Wire Line
 	1500 2100 1550 2100
-Wire Wire Line
-	1500 1900 1550 1900
-Wire Wire Line
-	1500 1600 1550 1600
-Wire Wire Line
-	1500 2000 1550 2000
 NoConn ~ 1550 1800
 Text GLabel 3000 1600 2    50   Input ~ 0
@@
 Text GLabel 3000 2500 2    50   Input ~ 0
 row_2
+Text GLabel 1500 1600 0    50   Input ~ 0
+row_1
 Text GLabel 3000 2600 2    50   Input ~ 0
-row_1
+col_15
 Text GLabel 3000 2700 2    50   Input ~ 0
-col_15
+col_14
 Text GLabel 2450 3150 3    50   Input ~ 0
-col_14
+col_13
 Text GLabel 2350 3150 3    50   Input ~ 0
-col_13
+col_12
 Text GLabel 2250 3150 3    50   Input ~ 0
-col_12
+col_11
 Text GLabel 2150 3150 3    50   Input ~ 0
-col_11
+col_10
 Text GLabel 2050 3150 3    50   Input ~ 0
-col_10
+col_9
 Text GLabel 1500 2700 0    50   Input ~ 0
-col_9
+col_8
 Text GLabel 1500 2600 0    50   Input ~ 0
-col_8
+col_7
 Text GLabel 1500 2500 0    50   Input ~ 0
-col_7
+col_6
 Text GLabel 1500 2400 0    50   Input ~ 0
-col_6
+col_5
 Text GLabel 1500 2300 0    50   Input ~ 0
-col_5
+col_4
 Text GLabel 1500 2200 0    50   Input ~ 0
-col_4
-Text GLabel 1500 2100 0    50   Input ~ 0
 col_3
-Text GLabel 1500 1600 0    50   Input ~ 0
+Text GLabel 1500 2000 0    50   Input ~ 0
 col_1
 Text GLabel 1500 1900 0    50   Input ~ 0
@@
 Wire Wire Line
 	2950 1800 3400 1800
-Text GLabel 1500 2000 0    50   Input ~ 0
+Text GLabel 1500 2100 0    50   Input ~ 0
 col_2
 Wire Wire Line
@@
 Wire Wire Line
 	10500 1850 10500 2600
+$Comp
+L GanJing_components:MX_1u_no_LED MX76
+U 1 1 61AD3FB4
+P 10250 1850
+F 0 "MX76" H 10300 1950 50  0000 C CNN
+F 1 "MX_1u_no_LED" H 10250 1850 50  0001 C CNN
+F 2 "GanJing_components:MX_1u_no_LED" H 10250 1850 50  0001 C CNN
+F 3 "https://datasheet.octopart.com/MX1A-11NW-Cherry-datasheet-34676.pdf" H 10250 1850 50  0001 C CNN
+F 4 "1u" H 10350 1700 50  0000 C CNN "Size"
+	1    10250 1850
+	1    0    0    -1
+$EndComp
+Wire Wire Line
+	10550 2050 10250 2050
+Connection ~ 10250 2050
+Wire Wire Line
+	10500 1850 10550 1850
+Wire Wire Line
+	2050 3150 2050 3100
 $EndSCHEMATC
