File: PCB/GanJing 65 rev 2.kicad_pcb (KiCad board)
At the start: 2 copper layers, 149 parts, among them SW1 EC11_rotary_encoder, U1 Elite-C

Commit message: Initial routing
Parts:
- moved D70 427.6 mm to (354.8, 176.2)
- moved D69 415.7 mm to (335.8, 176.2)
- moved D68 395.4 mm to (316.7, 176.2)
- moved D71 390.1 mm to (354.8, 140.5)
- moved D67 375.2 mm to (297.7, 176.2)
- moved D59 371.1 mm to (354.8, 159.5)
- moved D45 356.8 mm to (52.4, 157.2)
- moved D65 338.9 mm to (259.6, 176.2)
- moved D56 333.7 mm to (264.3, 157.2)
- moved D57 327.8 mm to (292.9, 157.2)
- moved D64 319.9 mm to (240.5, 176.2)
- moved D58 316.7 mm to (309.6, 131.0)
- moved D47 306.8 mm to (92.9, 157.2)
- moved D66 305.1 mm to (278.6, 176.2)
- moved D44 300.0 mm to (335.8, 159.5)
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Routing:
- net row_3: track 0.00 -> 313.8 mm
- net row_5: track 0.00 -> 310.0 mm
- net row_2: track 0.00 -> 298.3 mm
- net row_1: track 0.00 -> 281.0 mm
- net row_4: track 0.00 -> 280.8 mm
- net col_7: track 0.00 -> 158.9 mm
- net col_9: track 0.00 -> 108.7 mm
- net col_11: track 0.00 -> 108.7 mm
- net col_12: track 0.00 -> 108.7 mm
- net col_10: track 0.00 -> 108.7 mm
- net col_14: track 0.00 -> 102.3 mm
- net col_1: track 0.00 -> 101.0 mm
- net col_13: track 0.00 -> 99.0 mm
- net S1: track 0.00 -> 91.4 mm
- net col_3: track 0.00 -> 89.4 mm
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- added copper zone on B.Cu, net GND
- added copper zone on F.Cu, net GND
Other:
- board outline added: 323.9 x 95.2 mm

Commit message: Finished routing
Parts:
- added MX76: MX_1u_no_LED, GanJing_components:MX_1u_no_LED, F.Cu at (364.3, 142.9)
- moved DS1 0.24 mm to (354.8, 119.3)
Connections:
- U1 pad 1: col_1 -> row_1
- U1 pad 10: col_7 -> col_6
- U1 pad 11: col_8 -> col_7
- U1 pad 12: col_9 -> col_8
- U1 pad 13: S1 -> col_14
- U1 pad 14: row_1 -> S1
- U1 pad 25: col_10 -> col_9
- U1 pad 26: col_11 -> col_10
- U1 pad 27: col_12 -> col_11
- U1 pad 28: col_13 -> col_12
- U1 pad 29: col_14 -> col_13
- U1 pad 5: col_2 -> col_1
- U1 pad 6: col_3 -> col_2
- U1 pad 7: col_4 -> col_3
- U1 pad 8: col_5 -> col_4
- U1 pad 9: col_6 -> col_5
Routing:
- net col_1: track 101.0 -> 391.6 mm, vias 0 -> 1
- net col_2: track 87.5 -> 360.0 mm, vias 0 -> 1
- net col_3: track 89.4 -> 343.7 mm, vias 0 -> 1
- net col_4: track 67.5 -> 303.7 mm, vias 0 -> 1
- net col_5: track 67.5 -> 285.5 mm, vias 0 -> 1
- net col_6: track 67.5 -> 267.0 mm, vias 0 -> 1
- net col_7: track 158.9 -> 340.9 mm, vias 0 -> 1
- net col_8: track 67.5 -> 231.9 mm, vias 0 -> 1
- net col_9: track 108.7 -> 258.2 mm, vias 0 -> 1
- net col_10: track 108.7 -> 241.3 mm, vias 0 -> 1
- net row_4: track 280.8 -> 399.9 mm
- net col_11: track 108.7 -> 224.6 mm, vias 0 -> 1
- net row_1: track 281.0 -> 390.2 mm
- net col_12: track 108.7 -> 207.8 mm, vias 0 -> 1
- net col_13: track 99.0 -> 194.3 mm, vias 0 -> 1
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
Commit message: Adding images and optional key switch instead of rotory knob
Parts:
- moved D15 2.38 mm to (52.4, 119.1)
- moved D67 2.38 mm to (297.7, 178.6)
Routing:
- net row_2: track 342.2 -> 344.6 mm
- net Net-(D15-Pad2): track 5.85 -> 8.23 mm
- net row_5: track 385.6 -> 387.6 mm
- net Net-(D43-Pad2): track 36.0 -> 34.8 mm
- net col_7: track 340.9 -> 339.8 mm
- net col_11: track 224.6 -> 223.5 mm
- net col_12: track 207.8 -> 206.7 mm
- net col_10: track 241.3 -> 240.2 mm
- net col_9: track 258.2 -> 257.1 mm
- net col_8: track 231.9 -> 230.8 mm
- net row_4: track 399.9 -> 400.9 mm
- net Net-(D67-Pad2): track 5.85 -> 6.83 mm
- net GND: vias 97 -> 100
Other:
- board text added: "Designed by Mingze Jin"
