File: Case/Plate/GanJing 70 plate.kicad_pcb (KiCad board)
At the start: 2 copper layers, 330.8 x 102.2 mm, 0 parts

Commit message: Switching to KiCad 6.0.1 so some files have been converted and the component symbol library files has been converted from .lib to .kicad_sym
Other:
- net class Default removed

Commit message: Updating plate file
Other:
- board size 330.8 x 102.2 mm -> 324.8 x 104.2 mm
- board text added: "Designed by Mingze Jin"

Commit message: Updating case to 10mm boarders
Other:
- outline, holes or cut-outs redrawn
- board text removed: "Designed by Mingze Jin"

Commit message: Updating plate tolerances
Other:
- board size 324.8 x 104.2 mm -> 325.8 x 107.2 mm
