File: Case/Plate/GanJing 70 plate.kicad_pcb (KiCad board)
At the start: 2 copper layers, 325.8 x 107.2 mm, 0 parts

Commit message: Updating plate to support split shift key on the right side
Other:
- board size 325.8 x 107.2 mm -> 335.8 x 107.2 mm
